Commit message: solo12 model with microscopic feet

File: traj_generation/models/solo12_nofeet.urdf (robot description, URDF)
Before this commit: robot solo, 21 links, 20 joints
Links:
- link FL_FOOT: geometry collision sphere radius=0.0000001; visual sphere radius=0.0000001
- link FR_FOOT: geometry collision sphere radius=0.0000001; visual sphere radius=0.0000001
- link HL_FOOT: geometry collision sphere radius=0.0000001; visual sphere radius=0.0000001
- link HR_FOOT: geometry collision sphere radius=0.0000001; visual sphere radius=0.0000001
